File: Talkie/Hardware/talkie_module_1_0.brd (EAGLE design)
At the start: 49.2 x 99 mm, 21 parts, among them IC1 MEGA48/88/168-PU, IC2 4511N

Commit message: modified readme
Parts:
- added C3, C4: 100nF 50V, rcl:C025-025X050
- added R1, R3, R4, R5, R6, R7, R8, R9: 10k, SteveMarple:RES-AXIAL-0.4
- added S3, S4: TL36PO, switch:TL3XPO
- added U$6, U$8: J1, thonkiconn:THONKICONN
- moved S2 114.1 mm to (114.9, 26.7), turned to 90 degrees
- moved LED3 75.7 mm to (101.0, 26.7), turned to 270 degrees
- moved JP1 66.2 mm to (16.5, 33.7)
- moved U$1 63.2 mm to (24.1, 10.2)
- moved U$5 62.2 mm to (69.8, 10.2)
- moved JP3 60.5 mm to (3.17, 18.4), turned to 90 degrees
- moved RV5 56.7 mm to (69.8, 40.6), turned to 270 degrees
- moved IC2 56.1 mm to (102.9, 43.2), turned to 180 degrees
- moved U$3 55.3 mm to (54.6, 10.2)
- moved U$2 54.6 mm to (39.4, 10.2)
- moved R2 51.1 mm to (62.2, 36.2), turned to 270 degrees
- moved S1 42.1 mm to (85.1, 25.4), turned to 0 degrees
- moved C2 39.6 mm to (31.1, 35.6), turned to 90 degrees
- moved QF1 37.3 mm to (46.7, 39.0), turned to 270 degrees
- moved RV3 31.8 mm to (54.6, 40.6), turned to 270 degrees
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Connections:
- removed net 14: S2.3, S2.4
- removed net GND1: S2.1, S2.2
- new net N$10: LED3.7, R1.P$2
- new net N$11: LED3.5, R9.P$1
- new net N$15: IC2.12, R3.P$1
- new net N$16: LED3.6, R3.P$2
- new net N$17: IC2.11, R4.P$1
- new net N$18: LED3.4, R4.P$2
- new net N$19: IC2.10, R5.P$1
- new net N$20: LED3.2, R5.P$2
- new net N$21: IC2.9, R6.P$1
- new net N$22: LED3.1, R6.P$2
- new net N$23: IC2.15, R7.P$1
- new net N$24: LED3.9, R7.P$2
- new net N$25: IC2.14, R8.P$1
- new net N$26: LED3.10, R8.P$2
- new net N$27: C3.1, C4.1
- new net N$28: C3.2, C4.2
- new net N$8: IC2.13, R1.P$1
- new net N$9: U$8.P$3
- net 3: now also U$6.P$3
- net GND: now also U$6.P$1, U$8.P$1
Other:
- board size 49.2 x 99 mm -> 120 x 102 mm
