File: Mozzi/Hardware/Moz_Mo_1_1.brd (EAGLE design)
At the start: 108 x 39.4 mm, 35 parts, among them IC1 MCP2200, IC2 MEGA48/88/168-PU, J1 1503_12, J2 1503_12, J3 1503_12, J4 1503_12, U1 POWER, X1 USB, Y1 12MHz

Commit message: MozMo  opening Version 1_1 / Adding software folder
Parts:
- removed U1: POWER, eurorack:POWER_16
- added IC3: 78L05Z, linear:TO92
- added POWER: (no value), TomW:MA05-2
Connections:
- new net +12V: POWER.10, POWER.9
- new net -12V: POWER.1, POWER.2
- net +5V: no longer U1.11, U1.12
- net GND: now also POWER.3, POWER.4, POWER.5, POWER.6, POWER.7, POWER.8; no longer U1.3, U1.4, U1.5, U1.6, U1.7, U1.8
Routing:
- net +5V: track 148.6 -> 143.5 mm
Changed lines of the file:
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@@
 <class number="1" name="power" width="0.381" drill="0">
+</class>
+<class number="2" name="ground" width="0.6096" drill="0">
 </class>
 </classes>
@@
 </element>
 <element name="C1" library="SparkFun" package="CAP-PTH-SMALL" value="470n" x="101.6" y="19.05" smashed="yes" rot="R90">
-<attribute name="OC_FARNELL" value="1457660" x="101.6" y="19.05" size="1.778" layer="27" rot="R90" display="off"/>
+<attribute name="OC_FARNELL" value="1694347" x="101.6" y="19.05" size="1.778" layer="27" rot="R90" display="off"/>
 <attribute name="NAME" x="100.965" y="17.018" size="1.27" layer="25" rot="R90"/>
 </element>
@@
 <attribute name="OC_FARNELL" value="1340604" x="20.32" y="14.605" size="1.778" layer="27" rot="R270" display="off"/>
 </element>
-<element name="U1" library="eurorack" package="POWER_16" value="POWER" x="10.16" y="34.29" smashed="yes">
-<attribute name="OC_FARNELL" value="3418510" x="10.16" y="34.29" size="1.778" layer="27" display="off"/>
-</element>
 <element name="J4" library="og-lumberg" package="1503_12" value="1503_12" x="6.35" y="14.605" smashed="yes" rot="R270">
 <attribute name="OC_FARNELL" value="1340604" x="6.35" y="14.605" size="1.778" layer="27" rot="R270" display="off"/>
@@
 </element>
 <element name="U$3" library="Logo_jld" package="LOGO_HANABI" value="" x="0" y="2.54"/>
+<element name="IC3" library="linear" package="TO92" value="78L05Z" x="21.59" y="34.29"/>
+<element name="POWER" library="TomW" package="MA05-2" value="" x="8.89" y="34.29">
+<attribute name="OC_NEWARK" value="unknown" x="8.89" y="34.29" size="1.778" layer="27" display="off"/>
+<attribute name="MPN" value="" x="8.89" y="34.29" size="1.778" layer="27" display="off"/>
+<attribute name="MF" value="" x="8.89" y="34.29" size="1.778" layer="27" display="off"/>
+<attribute name="OC_FARNELL" value="unknown" x="8.89" y="34.29" size="1.778" layer="27" display="off"/>
+</element>
 </elements>
 <signals>
@@
 <contactref element="U$1" pad="P$3"/>
 <contactref element="U$2" pad="P$3"/>
-<contactref element="U1" pad="3"/>
-<contactref element="U1" pad="8"/>
-<contactref element="U1" pad="7"/>
-<contactref element="U1" pad="6"/>
-<contactref element="U1" pad="5"/>
-<contactref element="U1" pad="4"/>
 <contactref element="D3" pad="A"/>
 <contactref element="D4" pad="A"/>
@@
 <via x="100.33" y="36.195" extent="1-16" drill="0.6" shape="octagon"/>
 <via x="59.69" y="7.62" extent="1-16" drill="0.6" shape="octagon"/>
+<contactref element="POWER" pad="7"/>
+<contactref element="POWER" pad="5"/>
+<contactref element="POWER" pad="3"/>
+<contactref element="POWER" pad="4"/>
+<contactref element="POWER" pad="8"/>
+<contactref element="POWER" pad="6"/>
+<wire x1="100.33" y1="36.195" x2="103.759" y2="35.56" width="0" layer="19" extent="1-1"/>
+<wire x1="88.9" y1="29.21" x2="100.33" y2="36.195" width="0" layer="19" extent="1-1"/>
+<wire x1="98.425" y1="21.59" x2="88.9" y2="29.21" width="0" layer="19" extent="1-1"/>
+<wire x1="101.6" y1="19.05" x2="98.425" y2="21.59" width="0" layer="19" extent="1-1"/>
+<wire x1="100.31" y1="8.89" x2="101.6" y2="19.05" width="0" layer="19" extent="1-1"/>
+<wire x1="88.105" y1="10.16" x2="96.52" y2="5.08" width="0" layer="19" extent="16-16"/>
+<wire x1="87.63" y1="16.51" x2="88.105" y2="10.16" width="0" layer="19" extent="1-1"/>
+<wire x1="71.093" y1="15.24" x2="87.63" y2="16.51" width="0" layer="19" extent="1-1"/>
+<wire x1="67.785" y1="10.16" x2="71.093" y2="15.24" width="0" layer="19" extent="1-1"/>
+<wire x1="67.31" y1="20.32" x2="71.093" y2="15.24" width="0" layer="19" extent="1-1"/>
+<wire x1="64.77" y1="27.94" x2="67.31" y2="20.32" width="0" layer="19" extent="1-1"/>
+<wire x1="64.81" y1="34.29" x2="64.77" y2="27.94" width="0" layer="19" extent="1-1"/>
+<wire x1="59.69" y1="7.62" x2="67.785" y2="10.16" width="0" layer="19" extent="1-1"/>
+<wire x1="48.26" y1="1.905" x2="59.69" y2="7.62" width="0" layer="19" extent="1-1"/>
+<wire x1="34.29" y1="1.905" x2="48.26" y2="1.905" width="0" layer="19" extent="1-1"/>
+<wire x1="20.32" y1="1.905" x2="34.29" y2="1.905" width="0" layer="19" extent="1-1"/>
+<wire x1="6.35" y1="1.905" x2="20.32" y2="1.905" width="0" layer="19" extent="1-1"/>
+<wire x1="3.302" y1="24.003" x2="6.35" y2="1.905" width="0" layer="19" extent="1-1"/>
+<wire x1="17.78" y1="27.94" x2="3.302" y2="24.003" width="0" layer="19" extent="1-1"/>
+<wire x1="25.4" y1="27.94" x2="17.78" y2="27.94" width="0" layer="19" extent="1-1"/>
+<wire x1="33.02" y1="35.56" x2="25.4" y2="27.94" width="0" layer="19" extent="1-1"/>
+<wire x1="36.83" y1="27.94" x2="33.02" y2="35.56" width="0" layer="19" extent="1-1"/>
+<wire x1="6.35" y1="35.56" x2="6.35" y2="1.905" width="0" layer="19" extent="1-1"/>
+<wire x1="6.35" y1="33.02" x2="6.35" y2="35.56" width="0" layer="19" extent="1-1"/>
+<wire x1="8.89" y1="33.02" x2="6.35" y2="33.02" width="0" layer="19" extent="1-1"/>
+<wire x1="11.43" y1="33.02" x2="8.89" y2="33.02" width="0" layer="19" extent="1-1"/>
+<wire x1="8.89" y1="35.56" x2="6.35" y2="35.56" width="0" layer="19" extent="1-1"/>
+<wire x1="11.43" y1="35.56" x2="11.43" y2="33.02" width="0" layer="19" extent="1-1"/>
 </signal>
 <signal name="1(TX0)">
@@
 <contactref element="U$1" pad="P$1"/>
 <contactref element="U$2" pad="P$1"/>
-<contactref element="U1" pad="12"/>
-<contactref element="U1" pad="11"/>
 <contactref element="JP1" pad="1"/>
 <contactref element="JP2" pad="2"/>
@@
 <contactref element="D2" pad="C"/>
 <contactref element="D5" pad="C"/>
-<wire x1="16.51" y1="33.02" x2="16.51" y2="30.48" width="0.508" layer="1"/>
 <wire x1="16.51" y1="30.48" x2="13.97" y2="27.94" width="0.508" layer="1"/>
 <wire x1="27.94" y1="35.56" x2="26.035" y2="35.56" width="0.508" layer="1"/>
@@
 <wire x1="69.85" y1="29.21" x2="69.85" y2="27.94" width="0.508" layer="1"/>
 <wire x1="40.64" y1="30.48" x2="40.64" y2="27.94" width="0.508" layer="1"/>
-<wire x1="16.51" y1="35.56" x2="16.51" y2="33.02" width="0.508" layer="1"/>
 <wire x1="60.325" y1="31.75" x2="57.785" y2="34.29" width="0.508" layer="1"/>
 <wire x1="40.64" y1="30.48" x2="46.355" y2="36.195" width="0.508" layer="1"/>
@@
 <wire x1="6.35" y1="24.13" x2="6.35" y2="27.94" width="0.508" layer="16"/>
 </signal>
+<signal name="+12V" class="1">
+<contactref element="POWER" pad="9"/>
+<contactref element="POWER" pad="10"/>
+<wire x1="13.97" y1="35.56" x2="13.97" y2="33.02" width="0" layer="19" extent="1-1"/>
+</signal>
+<signal name="-12V" class="1">
+<contactref element="POWER" pad="1"/>
+<contactref element="POWER" pad="2"/>
+<wire x1="3.81" y1="35.56" x2="3.81" y2="33.02" width="0" layer="19" extent="1-1"/>
+</signal>
 </signals>
