File: Mozzi/Hardware/Moz_Mo_1_1.sch (EAGLE design)
At the start: 34 parts, among them IC1 MCP2200, IC2 MEGA48/88/168-PU, J1 1503_12, J2 1503_12, J3 1503_12, J4 1503_12, U1 POWER, X1 USB, Y1 12MHz

Commit message: MozMo  opening Version 1_1 / Adding software folder
Parts:
- removed U1: POWER, eurorack:POWER
- added IC3: 78L05Z, linear:78L05Z
- added POWER: (no value), TomW:10_PIN_HEADER
- C1: OC_FARNELL 1457660 -> 1694347
Connections:
- new net +12V: POWER.10, POWER.9
- new net -12V: POWER.1, POWER.2
- net +5V: no longer U1.+5V
- net GND: now also POWER.3, POWER.4, POWER.5, POWER.6, POWER.7, POWER.8; no longer U1.GND
Other:
- note added: "Power"
Changed lines of the file:
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@@
 <class number="1" name="power" width="0.381" drill="0">
+</class>
+<class number="2" name="ground" width="0.6096" drill="0">
 </class>
 </classes>
@@
 </part>
 <part name="C1" library="SparkFun" deviceset="CAP" device="PTH" value="470n">
-<attribute name="OC_FARNELL" value="1457660"/>
+<attribute name="OC_FARNELL" value="1694347"/>
 </part>
 <part name="C2" library="SparkFun" deviceset="CAP" device="PTH1" value="1u">
@@
 </part>
 <part name="GND8" library="SparkFun" deviceset="GND" device=""/>
-<part name="U1" library="eurorack" deviceset="POWER" device="">
-<attribute name="OC_FARNELL" value="3418510"/>
-</part>
 <part name="J4" library="og-lumberg" deviceset="1503_12" device="">
 <attribute name="OC_FARNELL" value="1340604"/>
@@
 <attribute name="OC_FARNELL" value="1227586"/>
 </part>
-<part name="GND11" library="SparkFun" deviceset="GND" device=""/>
-<part name="P+8" library="supply1" deviceset="+5V" device=""/>
 <part name="D3" library="SteveMarple" deviceset="DIODE-SCHOTTKY" device="" value="BAT85">
 <attribute name="OC_FARNELL" value="1612329"/>
@@
 </part>
 <part name="GND14" library="SparkFun" deviceset="GND" device=""/>
+<part name="IC3" library="linear" deviceset="78*" device="Z" technology="L05"/>
+<part name="POWER" library="TomW" deviceset="10_PIN_HEADER" device=""/>
 </parts>
 <sheets>
@@
 CC-BY-SA
 Jean-Luc Deladrière</text>
+<text x="132.08" y="68.58" size="1.778" layer="91">Power</text>
 </plain>
 <instances>
@@
 </instance>
 <instance part="GND8" gate="1" x="38.1" y="20.32"/>
-<instance part="U1" gate="G$1" x="157.48" y="81.28">
-<attribute name="OC_FARNELL" x="157.48" y="81.28" size="1.778" layer="96" display="off"/>
-</instance>
 <instance part="J4" gate="G$1" x="129.54" y="25.4">
 <attribute name="OC_FARNELL" x="129.54" y="25.4" size="1.778" layer="96" display="off"/>
@@
 <attribute name="KNOBFARNELL" x="132.08" y="152.4" size="1.778" layer="96" display="off"/>
 </instance>
-<instance part="GND11" gate="1" x="172.72" y="66.04"/>
-<instance part="P+8" gate="1" x="175.26" y="96.52"/>
 <instance part="D3" gate="G$1" x="30.48" y="68.58" rot="R90">
 <attribute name="OC_FARNELL" x="30.48" y="68.58" size="1.778" layer="96" rot="R90" display="off"/>
@@
 </instance>
 <instance part="GND14" gate="1" x="124.46" y="17.78"/>
+<instance part="IC3" gate="A1" x="127" y="88.9"/>
+<instance part="POWER" gate="G$1" x="134.62" y="53.34"/>
 </instances>
 <busses>
@@
 </segment>
 <segment>
-<pinref part="GND11" gate="1" pin="GND"/>
-<wire x1="172.72" y1="68.58" x2="172.72" y2="83.82" width="0.1524" layer="91"/>
-<wire x1="172.72" y1="83.82" x2="167.64" y2="83.82" width="0.1524" layer="91"/>
-<pinref part="U1" gate="G$1" pin="GND"/>
-</segment>
-<segment>
 <pinref part="C6" gate="G$1" pin="1"/>
 <pinref part="GND13" gate="1" pin="GND"/>
@@
 <pinref part="GND14" gate="1" pin="GND"/>
 <wire x1="124.46" y1="20.32" x2="124.46" y2="22.86" width="0.1524" layer="91"/>
+</segment>
+<segment>
+<pinref part="POWER" gate="G$1" pin="7"/>
+<wire x1="144.78" y1="55.88" x2="142.24" y2="55.88" width="0.1524" layer="91"/>
+<pinref part="POWER" gate="G$1" pin="5"/>
+<wire x1="144.78" y1="53.34" x2="142.24" y2="53.34" width="0.1524" layer="91"/>
+<wire x1="144.78" y1="55.88" x2="144.78" y2="53.34" width="0.1524" layer="91"/>
+<pinref part="POWER" gate="G$1" pin="3"/>
+<wire x1="144.78" y1="50.8" x2="142.24" y2="50.8" width="0.1524" layer="91"/>
+<wire x1="144.78" y1="53.34" x2="144.78" y2="50.8" width="0.1524" layer="91"/>
+<junction x="144.78" y="53.34"/>
+<label x="147.32" y="53.34" size="1.778" layer="95"/>
+</segment>
+<segment>
+<pinref part="POWER" gate="G$1" pin="4"/>
+<wire x1="124.46" y1="50.8" x2="127" y2="50.8" width="0.1524" layer="91"/>
+<pinref part="POWER" gate="G$1" pin="8"/>
+<wire x1="124.46" y1="55.88" x2="127" y2="55.88" width="0.1524" layer="91"/>
+<wire x1="124.46" y1="50.8" x2="124.46" y2="53.34" width="0.1524" layer="91"/>
+<pinref part="POWER" gate="G$1" pin="6"/>
+<wire x1="124.46" y1="53.34" x2="124.46" y2="55.88" width="0.1524" layer="91"/>
+<wire x1="124.46" y1="53.34" x2="127" y2="53.34" width="0.1524" layer="91"/>
+<junction x="124.46" y="53.34"/>
+<label x="119.38" y="53.34" size="1.778" layer="95"/>
 </segment>
 </net>
@@
 <wire x1="132.08" y1="127" x2="132.08" y2="124.46" width="0.1524" layer="91"/>
 <pinref part="P+6" gate="1" pin="+5V"/>
-</segment>
-<segment>
-<pinref part="P+8" gate="1" pin="+5V"/>
-<wire x1="175.26" y1="93.98" x2="175.26" y2="78.74" width="0.1524" layer="91"/>
-<wire x1="175.26" y1="78.74" x2="167.64" y2="78.74" width="0.1524" layer="91"/>
-<pinref part="U1" gate="G$1" pin="+5V"/>
 </segment>
 <segment>
@@
 </segment>
 </net>
+<net name="+12V" class="1">
+<segment>
+<pinref part="POWER" gate="G$1" pin="9"/>
+<wire x1="144.78" y1="58.42" x2="142.24" y2="58.42" width="0.1524" layer="91"/>
+<label x="144.78" y="58.42" size="1.778" layer="95"/>
+</segment>
+<segment>
+<pinref part="POWER" gate="G$1" pin="10"/>
+<wire x1="124.46" y1="58.42" x2="127" y2="58.42" width="0.1524" layer="91"/>
+<label x="119.38" y="58.42" size="1.778" layer="95"/>
+</segment>
+</net>
+<net name="-12V" class="1">
+<segment>
+<pinref part="POWER" gate="G$1" pin="1"/>
+<wire x1="142.24" y1="48.26" x2="144.78" y2="48.26" width="0.1524" layer="91"/>
+<label x="147.32" y="48.26" size="1.778" layer="95"/>
+</segment>
+<segment>
+<pinref part="POWER" gate="G$1" pin="2"/>
+<wire x1="124.46" y1="48.26" x2="127" y2="48.26" width="0.1524" layer="91"/>
+<label x="119.38" y="48.26" size="1.778" layer="95"/>
+</segment>
+</net>
