File: Talko/Hardware/Talko_1_0.brd (EAGLE design)
At the start: 50 x 105 mm, 59 parts, among them IC1 MEGA8-AI, IC2 4511D, IC5 MCP2200, J1 AVR_SPI, Q1 16 MHz, X3 USB

Commit message: Fixing a bug in loop mode changing switch reference @ Mouser (for a bigger lever)
Parts:
- C9: value 22u -> 10u
- R10: value 100K -> 10K
