File: Talko/Hardware/Talko_1_1.brd (EAGLE design)
At the start: 50 x 105 mm, 56 parts, among them IC1 MEGA8-AI, IC2 4511D, IC5 MCP2200, J1 AVR_SPI, Q1 16 MHz, X3 USB

Commit message: renaming Talko pots on v1.1
Parts:
- R3: value 4470R -> 470R
- R9: value 390R -> 470R
- flipped JP1 to the bottom, turned to 270 degrees
- renumbered CV to SOUND, RV1 to SOUND_POT, RV2 to PITCH_POT, RV3 to SPEED_POT, RV4 to BEND_POT
Routing:
- net VUSB: vias 0 -> 2
- net +5V: vias 3 -> 4
Other:
- board text added: "Talko 1.1"
- board text added: "usb+5V"
- board text removed: "Talko 1.0"
- board text removed: "usb +5V"
